File: IC101.sch (KiCad schematic (older format))
At the start: 36 parts

Commit message: Some rearrangements/
Connections:
- net BLB renamed BLB-1
- net BLG renamed BLG-6
- net BLR renamed BLR-11
- net Bin renamed Bin-2
- net Bout renamed Bout-4
- net Gin renamed Gin-7
- net Gout renamed Gout-9
- net Rin renamed Rin-12
- net Rout renamed Rout-14
Changed lines of the file:
@@
 encoding utf-8
 Sheet 5 6
-Title "NANAO MS8-29"
-Date "2025-10-10"
-Rev "1.5"
+Title "NANAO MS8-29 (05A00362G1)"
+Date "2025-11-17"
+Rev "1.6"
 Comp "Franck BOURDONNEC"
 Comment1 ""
@@
 	5250 2850 8100 2850
 Text HLabel 9250 2850 2    50   Output ~ 0
-Gout
+Gout-9
 $Comp
 L Device:R R111
@@
 	4650 2500 4650 2650
 Text HLabel 1400 4050 0    50   Input ~ 0
-Gin
+Gin-7
 $Comp
 L Transistor_BJT:MMBT3904 Q?
@@
 	3450 2250 8100 2250
 Text HLabel 9250 2250 2    50   Output ~ 0
-Rout
+Rout-14
 Wire Wire Line
 	2850 1750 2850 1900
@@
 Wire Wire Line
 	2850 1350 3450 1350
-Text HLabel 1400 3850 0    50   Input ~ 0
-Rin
+Text HLabel 1450 3850 0    50   Input ~ 0
+Rin-12
 $Comp
 L Device:R R121
@@
 $EndComp
 Text HLabel 1400 4250 0    50   Input ~ 0
-Bin
+Bin-2
 Text HLabel 9250 3450 2    50   Output ~ 0
-Bout
+Bout-4
 Connection ~ 7100 3450
 Wire Wire Line
@@
 Wire Wire Line
 	1100 1350 2500 1350
-Text HLabel 1400 2250 0    50   Input ~ 0
-BLR
-Text HLabel 1400 2850 0    50   Input ~ 0
-BLG
-Text HLabel 1400 3450 0    50   Input ~ 0
-BLB
+Text HLabel 1500 2250 0    50   Input ~ 0
+BLR-11
+Text HLabel 1450 2850 0    50   Input ~ 0
+BLG-6
+Text HLabel 1450 3450 0    50   Input ~ 0
+BLB-1
 Text Notes 1200 2200 0    50   ~ 0
 Blacks levels setup
@@
 $EndComp
 Wire Wire Line
-	1850 3850 1400 3850
+	1850 3850 1450 3850
 $Comp
 L Device:R R?
@@
 	5800 5400 5800 5750
 Wire Wire Line
-	1400 2250 2500 2250
-Wire Wire Line
-	1400 2850 4300 2850
-Wire Wire Line
-	1400 3450 6150 3450
+	1500 2250 2500 2250
+Wire Wire Line
+	1450 2850 4300 2850
+Wire Wire Line
+	1450 3450 6150 3450
 Wire Wire Line
 	7100 5750 6500 5750
