File: IC101.sch (KiCad schematic (older format))
At the start: 36 parts

Commit message: Some corrections
Parts:
- Cx1, Cx2, Cx3: renamed from C?; value C -> 1n; footprint (none) -> Capacitor_SMD:C_0805_2012Metric_Pad1.18x1.45mm_HandSolder; LCSC (none) -> C46653
- Qx1, Qx2, Qx3, Qx4, Qx5, Qx6: renamed from Q?; LCSC (none) -> C20526
- Rx1, Rx2, Rx3: renamed from R?; footprint (none) -> Resistor_SMD:R_0805_2012Metric_Pad1.20x1.40mm_HandSolder; LCSC (none) -> C326608
- Rx10, Rx12, Rx15, Rx17, Rx5, Rx7: renamed from R?; footprint (none) -> Resistor_SMD:R_0805_2012Metric_Pad1.20x1.40mm_HandSolder; LCSC (none) -> C17798
- Rx11, Rx16, Rx6: renamed from R?; footprint (none) -> Resistor_SMD:R_0805_2012Metric_Pad1.20x1.40mm_HandSolder; LCSC (none) -> C4310
- Rx13, Rx18, Rx8: renamed from R?; footprint (none) -> Resistor_SMD:R_0805_2012Metric_Pad1.20x1.40mm_HandSolder; LCSC (none) -> C17513
- Rx14, Rx4, Rx9: renamed from R?; footprint (none) -> Resistor_SMD:R_0805_2012Metric_Pad1.20x1.40mm_HandSolder; LCSC (none) -> C26010
- Rx19, Rx20, Rx21: renamed from R?; footprint (none) -> Resistor_SMD:R_0805_2012Metric_Pad1.20x1.40mm_HandSolder; LCSC (none) -> C17714
Connections:
- net BLB-1: no longer R121.1
- net BLG-6: no longer R111.1
- net BLR-11: no longer R101.1
- net GND10: no longer Qx2.3 (C), Qx4.3 (C), Qx6.3 (C), Rx11.1, Rx14.1, Rx16.1, Rx4.1, Rx6.1, Rx9.1
- net at Qx3.2 (E), Rx12.2, Rx2.1: now also R111.1
- net at Qx5.2 (E), Rx17.2, Rx3.1: now also R121.1
- net at Qx1.2 (E), Rx1.1, Rx7.2: now also R101.1
- new net VCC15: Qx2.3 (C), Qx4.3 (C), Qx6.3 (C), Rx11.1, Rx14.1, Rx16.1, Rx4.1, Rx6.1, Rx9.1
Other:
- note added: "I added some identification labels for the components\nto help identify them on my repro of the four small PCB.\n\nIt's a set of IC101, IC102, IC103 and IC402 populated with\nall cms components when available.\n\nContact me if you need a set."
