File: IC102.sch (KiCad schematic (older format))
At the start: 26 parts

Commit message: Some corrections
Parts:
- C1: renamed from __C1; footprint (none) -> Capacitor_SMD:C_0805_2012Metric_Pad1.18x1.45mm_HandSolder; LCSC (none) -> C1710
- C2: renamed from __C2; footprint (none) -> Capacitor_SMD:C_0805_2012Metric_Pad1.18x1.45mm_HandSolder; LCSC (none) -> C1743
- C3: footprint (none) -> Capacitor_SMD:C_0805_2012Metric_Pad1.18x1.45mm_HandSolder; LCSC (none) -> C46653
- C4: renamed from __C4; footprint (none) -> Capacitor_SMD:C_0805_2012Metric_Pad1.18x1.45mm_HandSolder; LCSC (none) -> C1754
- C5: renamed from __C5; footprint (none) -> Capacitor_SMD:C_0805_2012Metric_Pad1.18x1.45mm_HandSolder; LCSC (none) -> C1790
- C6: renamed from __C6; footprint (none) -> Capacitor_SMD:C_0805_2012Metric_Pad1.18x1.45mm_HandSolder; LCSC (none) -> C107145
- D1: renamed from __D1; value D -> 4148; footprint (none) -> Diode_SMD:D_SOD-323_HandSoldering; LCSC (none) -> C2128
- D2: renamed from __D?; value D -> 4148; footprint (none) -> Diode_SMD:D_SOD-323_HandSoldering; LCSC (none) -> C2128
- Q1: renamed from __Q1; LCSC (none) -> C20526
- Q2: renamed from __Q2; LCSC (none) -> C20526
- Q3: renamed from __Q3; LCSC (none) -> C20526
- Q4: renamed from __Q4; LCSC (none) -> C2143
- R1: renamed from __R?; footprint (none) -> Resistor_SMD:R_0805_2012Metric_Pad1.20x1.40mm_HandSolder; LCSC (none) -> C17444
- R10: renamed from __R10; footprint (none) -> Resistor_SMD:R_0805_2012Metric_Pad1.20x1.40mm_HandSolder; LCSC (none) -> C17713
- R11: renamed from __R11; footprint (none) -> Resistor_SMD:R_0805_2012Metric_Pad1.20x1.40mm_HandSolder; LCSC (none) -> C149504
- R13: renamed from __R13; footprint (none) -> Resistor_SMD:R_0805_2012Metric_Pad1.20x1.40mm_HandSolder; LCSC (none) -> C17513
- R14: renamed from __R14; footprint (none) -> Resistor_SMD:R_0805_2012Metric_Pad1.20x1.40mm_HandSolder; LCSC (none) -> C17709
- R15: renamed from __R15; footprint (none) -> Resistor_SMD:R_0805_2012Metric_Pad1.20x1.40mm_HandSolder; LCSC (none) -> C17593
- R2: renamed from __R2; footprint (none) -> Resistor_SMD:R_0805_2012Metric_Pad1.20x1.40mm_HandSolder; LCSC (none) -> C17560
- R3: renamed from __R3; footprint (none) -> Resistor_SMD:R_0805_2012Metric_Pad1.20x1.40mm_HandSolder; LCSC (none) -> C17801
- R4: renamed from __R4; footprint (none) -> Resistor_SMD:R_0805_2012Metric_Pad1.20x1.40mm_HandSolder; LCSC (none) -> C17520
- R5: renamed from __R5; footprint (none) -> Resistor_SMD:R_0805_2012Metric_Pad1.20x1.40mm_HandSolder; LCSC (none) -> C17614
- R6: renamed from __R6; footprint (none) -> Resistor_SMD:R_0805_2012Metric_Pad1.20x1.40mm_HandSolder; LCSC (none) -> C17713
- R7: renamed from __R7; footprint (none) -> Resistor_SMD:R_0805_2012Metric_Pad1.20x1.40mm_HandSolder; LCSC (none) -> C17560
- R8: renamed from __R8; footprint (none) -> Resistor_SMD:R_0805_2012Metric_Pad1.20x1.40mm_HandSolder
- R9: renamed from __R9; footprint (none) -> Resistor_SMD:R_0805_2012Metric_Pad1.20x1.40mm_HandSolder; LCSC (none) -> C17560
Other:
- note added: "LSCS 10n"
- note added: "LSCS 220pF"
