File: nanao-ms8-29.sch (KiCad schematic (older format))
At the start: 453 parts, among them CN101 JST JH, CN102 Conn_01x08_Male, CN103 B10B_PH-K-S, CN104 Conn_01x11_Male, CN105 B14B_PH-K-S, CN106 Conn_01x14_Male, CN302 JST JH, CN303 Conn_01x05_Female, CN402 Conn_01x02_Female, CN570 Conn_01x05_Male, CN808 Degauss, CN901 B2P3-VH, CN902 Conn_01x02_Female, CN903 Conn_01x05_Female, IC101-1 SHIC101, IC102 SHIC102, IC103 SHIC103, IC401 LA7830, Q301 2SC1740, Q302 2SC1044, Q303 2SC4218, Q304 2SA1624, Q305 DTD113ES, Q311 2SC1740, Q312 2SC1044, Q313 2SC4218, Q314 2SA1624, Q315 DTD113ES, Q321 2SC1740, Q322 2SC1044, Q323 2SC4218, Q324 2SA1624, Q325 DTD113ES, Q401 2SC3621, Q402 2SA1408, Q404 2SA1091, Q405 2SA933, Q408 2SC3621, Q521 2SC1740, Q530 2SA933, Q531 2SC1740, Q532 2SC2688, Q533 2SC3998, Q535 2SA933, Q560 2SA1091, Q561 2SC2705, Q570 2SA1091, Q571 2SA1091, Q572 2SA966, Q901 2SC3306 BUW13A, Q902 2SA1091, Q903 2SC2482, Q904 2SC2655, SW501 SW2inv, SW502 SW_SPDT, T530 ETH19Y141AY, T531 EHT, T901 5F13121B1B

Commit message: Add files via upload
Rework degauss/power section
Parts:
- removed CN902: Conn_01x02_Female, symbol Connector:Conn_01x02_Female
- removed R801: 903051D050MP, symbol Device:Thermistor_PTC_3wire
- added PTH901: degauss-pth, symbol nanao:degauss-pth
- BR901: value DBF60E -> BF40E2; symbol Device:D_Bridge_+-AA -> Device:D_Bridge_+AA-
- CN901: symbol Connector:Conn_01x02_Female -> Connector:Conn_01x03_Female
- F901: value 250v 3 -> 250v 3A
- xCN901: symbol Connector:Conn_01x02_Male -> Connector:Conn_01x03_Male
- renumbered C903 to C902, C902 to C903, C916 to C915, C915 to C916, CN808 to CN902
Connections:
- wire segments 1307 -> 1302
- no-connect marks 7 -> 9
Other:
- note added: "check this harness"
- note removed: "check this wiring"
- moved on the sheet: C915, C916, CN902, F901, NTH901, R901

Commit message: Fixe some values
Parts:
- C550, C551: value 270n/100v -> 2µ7/100v
- C554: value 330n/200v -> 390n/200v
- R541: value 2K7 -> 27
- VR434: value 5K -> 30K
Other:
- note added: "Components to check values:\nR442 1K2 2K2 ?\nC554 270n 390n ?\n"
Changed lines of the file:
@@
 Title "NANAO MS8-29"
 Date "2025-04-10"
-Rev "1.2"
+Rev "1.3"
 Comp "Franck BOURDONNEC"
 Comment1 ""
@@
 U 1 1 6F7ACC93
 P 5700 8200
-F 0 "VR431" H 5550 8050 50  0000 C CNN
-F 1 "5K" H 5550 8250 50  0000 C CNN
+F 0 "VR431" H 6050 8250 50  0000 C CNN
+F 1 "5K" H 6000 8150 50  0000 C CNN
 F 2 "" H 5700 8200 50  0001 C CNN
 F 3 "~" H 5700 8200 50  0001 C CNN
@@
 P 17000 15250
 F 0 "C550" H 17000 15350 50  0000 L CNN
-F 1 "270n/100v" V 16950 14750 50  0000 L CNN
+F 1 "2µ7/100v" V 16950 14750 50  0000 L CNN
 F 2 "" H 17038 15100 50  0001 C CNN
 F 3 "~" H 17000 15250 50  0001 C CNN
@@
 P 18050 12850
 F 0 "C554" H 17850 12950 50  0000 L CNN
-F 1 "330n/200v" V 18150 12650 50  0000 L CNN
+F 1 "390n/200v" V 18150 12650 50  0000 L CNN
 F 2 "" H 18088 12700 50  0001 C CNN
 F 3 "~" H 18050 12850 50  0001 C CNN
@@
 P 7300 10700
 F 0 "VR434" H 7100 10650 50  0000 C CNN
-F 1 "5K" H 7150 10750 50  0000 C CNN
+F 1 "30K" H 7150 10750 50  0000 C CNN
 F 2 "" H 7300 10700 50  0001 C CNN
 F 3 "~" H 7300 10700 50  0001 C CNN
@@
 P 16750 15250
 F 0 "C551" H 16750 15350 50  0000 L CNN
-F 1 "270n/100v" V 16700 14750 50  0000 L CNN
+F 1 "2µ7/100v" V 16700 14750 50  0000 L CNN
 F 2 "" H 16788 15100 50  0001 C CNN
 F 3 "~" H 16750 15250 50  0001 C CNN
@@
 P 14000 13400
 F 0 "R541" H 13850 13350 50  0000 C CNN
-F 1 "2K7" H 13850 13450 50  0000 C CNN
+F 1 "27" H 13850 13450 50  0000 C CNN
 F 2 "" V 13930 13400 50  0001 C CNN
 F 3 "~" H 14000 13400 50  0001 C CNN
@@
 Wire Wire Line
 	4700 15700 4950 15700
+Text Notes 21400 13950 0    50   ~ 0
+Components to check values:\nR442   1K2 2K2 ?\nC554   270n 390n ?\n
 $EndSCHEMATC

Commit message: Add files via upload
Redraw some parts, try to be consistent with ref/values positioning.
Fix an error around C542
Parts:
- F902: value 125v 2A -> 2A
- R446: value 68K/ .5W -> 68K 1/2W
- R551: value 2K7 -> 2K7 / 4W
- TP21: value N -> Narrow
- TP42: value W -> Wide
- Tube1: value CRT -> A68KJU96X
- renumbered R415 to R913
Connections:
- net labels added: 12.5v, 94v, E1524
- net labels removed: 0.46v, 1v, 6.42v, 93.3v, ?, E, GND1, SS
- wire segments 1302 -> 1276
- no-connect marks 9 -> 10
Other:
- note added: "ALTERNATES (tested OK)\n2SC4288A Toshiba\nBU2532AL Philips"
- note added: "I have an extra\n1µ/630v on\nC548\n"
- note added: "MSU1FGS514\nHR46598"
- note added: "Make R542 2W"
- note added: "Metalized caps\nself healing"
- note added: "focus sharpener"
- note added: "low plugged in"
- note removed: "9x Metalized caps\nself healing"
- note removed: "Components to check values:\nR442 1K2 2K2 ?\nC554 270n 390n ?\n"
- note removed: "x"
- moved on the sheet: C406, C520, C521, C534, C536, C540, C541, C542, C543, C544, C545, C546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

Commit message: Add files via upload
Some corrections
+Buymecoffee ;)
Parts:
- added D305, D315, D325: 1SS244, Diode_THT:D_DO-41_SOD81_P10.16mm_Horizontal, symbol Diode:1N4007
- added R307: 1K, symbol Device:R
- C446: value 4µ7NP -> 33µ BP 16v
- L301, L311, L321: value 10µH -> 22µH
- L302, L312, L322: value 1µH -> 1µ8H
- L570: value 22µH -> 100µH
- R302, R312, R322: value 68 -> 33
- R303, R313, R323: value 62K -> 220K
- R307, R317, R327: value 270, 1/2W -> 270, 2W
- SG301, SG311, SG321, SG331, SG332: value SPARK_GAP -> 1Kv
Connections:
- wire segments 1276 -> 1289
Other:
- note removed: "FLAMEPROOF LIST\n(fuse résistors)\n"
- note removed: "POLARIZED CAPS\n\n\n(T : tantalum)\ndefault size 5mm diam,\n5mm pitch"
- moved on the sheet: C302, C431, C434, C436, CN402, R303, R304, R435, ZD301

Commit message: Some rearrangements/
Parts:
- CN103: value B10B_PH-K-S -> B11B_PH-K-S
- renumbered ZD121 to ZD101, ZD101 to ZD121
Connections:
- wire segments 1289 -> 1284
Other:
- note added: "+12v"
- note added: "C433 is 1n on every datasheet\nof the 783x serie.\nSome comments says replace it (with R433) when\nframe foldover. So add it !, pcb have correct traces."
- moved on the sheet: C402, C405, C579, R588, ZD101, ZD121

Commit message: IC401 is LA7832 not LA7830
Parts:
- IC401: value LA7830 -> LA7832
Other:
- note added: "BL+"
Changed lines of the file:
@@
 Sheet 1 6
 Title "NANAO MS8-29 (05A00362G1)"
-Date "2025-11-17"
-Rev "1.6"
+Date "2026-01-30"
+Rev "1.6a"
 Comp "Franck BOURDONNEC"
 Comment1 ""
@@
 P 10000 8450
 F 0 "IC401" H 9650 8900 50  0000 L CNN
-F 1 "LA7830" H 9250 8900 50  0000 L CNN
+F 1 "LA7832" H 9250 8900 50  0000 L CNN
 F 2 "" H 10000 8450 50  0001 C CNN
 F 3 "" H 10000 8450 50  0001 C CNN
@@
 	11400 14800 11400 14750
 Text Notes 13850 11400 0    157  ~ 31
-B+
+BL+
 Text Notes 17650 9750 0    157  ~ 31
 B+
