File: nanao-ms8-29.sch (KiCad schematic (older format))
At the start: 456 parts, among them CN101 JST JH, CN102 Conn_01x08_Male, CN103 B11B_PH-K-S, CN104 Conn_01x11_Male, CN105 B14B_PH-K-S, CN106 Conn_01x14_Male, CN302 JST JH, CN303 Conn_01x05_Female, CN402 Conn_01x02_Female, CN570 Conn_01x05_Male, CN901 B2P3-VH, CN902 Degauss, CN903 Conn_01x05_Female, IC101-1 SHIC101, IC102 SHIC102, IC103 SHIC103, IC401 LA7832, Q301 2SC1740, Q302 2SC1044, Q303 2SC4218, Q304 2SA1624, Q305 DTD113ES, Q311 2SC1740, Q312 2SC1044, Q313 2SC4218, Q314 2SA1624, Q315 DTD113ES, Q321 2SC1740, Q322 2SC1044, Q323 2SC4218, Q324 2SA1624, Q325 DTD113ES, Q401 2SC3621, Q402 2SA1408, Q404 2SA1091, Q405 2SA933, Q408 2SC3621, Q521 2SC1740, Q530 2SA933, Q531 2SC1740, Q532 2SC2688, Q533 2SC3998, Q535 2SA933, Q560 2SA1091, Q561 2SC2705, Q570 2SA1091, Q571 2SA1091, Q572 2SA966, Q901 2SC3306 BUW13A, Q902 2SA1091, Q903 2SC2482, Q904 2SC2655, SW501 SW2inv, SW502 SW_SPDT, T530 ETH19Y141AY, T531 EHT, T901 5F13121B1B

Commit message: Some corrections
Parts:
- added R467: 2K2, symbol Device:R
- C447: value 470/25v -> 47/25v
Connections:
- net labels added: 18v
- wire segments 1284 -> 1291
Other:
- note added: "330 or 470 \nor 500 on R564"
- note added: "94v"
- note added: "ALTERNATES (tested OK)\n2SC4288A Toshiba\nBU2532AL Philips\nFJL6920 Onsemi"
- note added: "Equivalence\nQ303, Q313, Q323 = 2SC2482\nQ304, Q314, Q324 = 2SA1091\n\nD305, D315, D325 only on ms9-29 !\n"
- note added: "This \nstage (R545..C533)\nmaybe unpopulated"
- note removed: "330 sur R564"
- note removed: "ALTERNATES (tested OK)\n2SC4288A Toshiba\nBU2532AL Philips"
- moved on the sheet: C446, C534, D305, D315, D325, NTH401, R433, R454, R463, R465, R466, R468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
