File: Notes.sch (KiCad schematic (older format))
At the start: 0 parts

Commit message: Some corrections
Other:
- note added: "TIPS:\n===\n\nNo Hsync at 15KHz:\nC913 is draining down the 12v to 6v.\nThis makes the HA11423 do 24KHz.\nIf you put the plug to 24KHz, the HOT\nfries directly (36KHz).\n\nWhitout the HOT installed, there is not enough\njuice through TH901 to produce a correct 18v and 12v !\n\n\nProblems with pincushion: reflow IC401 ON THE VERTICAL BOARD."
- note added: "V1.6a\n\nIC401 is LA7832 not LA7830\n\nI installed a FJL6920. Works OK.\nhttps://www.arcadepartsandrepair.com/store/integrated-circuits/transistors/fjl6920-high-output-transistor/"
- note added: "V1.7\n\nMeasured caps on SHIC101 ( 1n )\nAdd identification on ICxxx for making the 4 pcb.\n\nAdded R467 around Hsize and redraw schematic.\n\nAdded some equivalent (tested) TR ref, for neckboard.\n\nnote on R545..C533 not always populated\n\nC447 is 47µ not 470µ"
- note removed: "V1.6a\n\nIC401 is LA7832 not LA7830"
Changed lines of the file:
@@
 Sheet 6 6
 Title "NANAO MS8-29 (05A00362G1)"
-Date "2026-01-30"
-Rev "1.6a"
+Date "2026-08-29"
+Rev "1.7"
 Comp "Franck BOURDONNEC"
 Comment1 ""
@@
 V1.6\n\nRework IC102
 Text Notes 3350 1600 0    50   ~ 0
-V1.6a\n\nIC401 is LA7832 not LA7830
+V1.6a\n\nIC401 is LA7832 not LA7830\n\nI installed a FJL6920. Works OK.\nhttps://www.arcadepartsandrepair.com/store/integrated-circuits/transistors/fjl6920-high-output-transistor/
+Text Notes 3350 2750 0    50   ~ 0
+V1.7\n\nMeasured caps on SHIC101 ( 1n )\nAdd identification on ICxxx for making the 4 pcb.\n\nAdded R467 around Hsize and redraw schematic.\n\nAdded some equivalent (tested) TR ref, for neckboard.\n\nnote on R545..C533 not always populated\n\nC447 is 47µ not 470µ
+Text Notes 1150 4750 0    50   ~ 0
+TIPS:\n===\n\nNo Hsync at 15KHz:\nC913 is draining down the 12v to 6v.\nThis makes the HA11423 do 24KHz.\nIf you put the plug to 24KHz, the HOT\nfries directly (36KHz).\n\nWhitout the HOT installed, there is not enough\njuice through TH901 to produce a correct 18v and 12v !\n\n\nProblems with pincushion: reflow IC401 ON THE VERTICAL BOARD.
 $EndSCHEMATC
