File: SHIC103.sch (KiCad schematic (older format))
At the start: 13 parts

Commit message: Some corrections
Parts:
- added C533b1: 5n6, Capacitor_THT:C_Rect_L7.0mm_W3.5mm_P2.50mm_P5.00mm, symbol Device:C
- added TP1: GND, TestPoint:TestPoint_Bridge_Pitch2.54mm_Drill1.0mm, symbol Connector:TestPoint
- added TP2: H, TestPoint:TestPoint_Bridge_Pitch2.54mm_Drill1.0mm, symbol Connector:TestPoint
- added TP3: V, TestPoint:TestPoint_Bridge_Pitch2.54mm_Drill1.0mm, symbol Connector:TestPoint
- C420: renamed from C_420; footprint (none) -> Capacitor_THT:CP_Radial_D4.0mm_P2.00mm
- C421: renamed from C_421; footprint (none) -> Capacitor_SMD:C_0805_2012Metric_Pad1.18x1.45mm_HandSolder; LCSC (none) -> C1755
- C430: renamed from C_430; footprint (none) -> Capacitor_THT:CP_Radial_D4.0mm_P2.00mm
- C530: renamed from C_530; footprint (none) -> Capacitor_SMD:C_0805_2012Metric_Pad1.18x1.45mm_HandSolder; LCSC (none) -> C1710
- C531: renamed from C_531; footprint (none) -> Capacitor_SMD:C_0805_2012Metric_Pad1.18x1.45mm_HandSolder; LCSC (none) -> C1755
- C532: renamed from C_532; footprint (none) -> Capacitor_THT:CP_Radial_D4.0mm_P2.00mm
- C533: renamed from C_533; footprint (none) -> Capacitor_SMD:C_0805_2012Metric_Pad1.18x1.45mm_HandSolder; LCSC (none) -> C113862
- IC502: renamed from IC_502; footprint (none) -> _my:HA11423
- R422: renamed from R_422; footprint (none) -> Resistor_SMD:R_0805_2012Metric_Pad1.20x1.40mm_HandSolder; LCSC (none) -> C17828
- R430: renamed from R_430; footprint (none) -> Resistor_SMD:R_0805_2012Metric_Pad1.20x1.40mm_HandSolder; LCSC (none) -> C17575
- R432: renamed from R_432; footprint (none) -> Resistor_SMD:R_0805_2012Metric_Pad1.20x1.40mm_HandSolder; LCSC (none) -> C110574
- R531: renamed from R_531; footprint (none) -> Resistor_SMD:R_0805_2012Metric_Pad1.20x1.40mm_HandSolder; LCSC (none) -> C17801
- R532: renamed from R_532; footprint (none) -> Resistor_SMD:R_0805_2012Metric_Pad1.20x1.40mm_HandSolder; LCSC (none) -> C17772
Connections:
- net GND: now also C533b1.2, TP1.1
- net pin11_hdrv: now also TP2.1
- net pin13_hhold: now also C533b1.1
- net pin7_vdrv: now also TP3.1
Changed lines of the file:
@@
 Sheet 4 6
 Title "NANAO MS8-29 (05A00362G1)"
-Date "2026-01-30"
-Rev "1.6a"
+Date "2026-08-29"
+Rev "1.7"
 Comp "Franck BOURDONNEC"
 Comment1 ""
@@
 $EndDescr
 $Comp
-L nanao:HA11423 IC_502
+L nanao:HA11423 IC502
 U 1 1 AA7324CA
 P 8100 3850
-F 0 "IC_502" H 10744 3896 50  0000 L CNN
-F 1 "HA11423" H 10744 3805 50  0000 L CNN
-F 2 "" H 8500 4150 50  0001 C CNN
+F 0 "IC502" H 5600 4900 50  0000 L CNN
+F 1 "HA11423" H 10050 4900 50  0000 L CNN
+F 2 "_my:HA11423" H 8500 4150 50  0001 C CNN
 F 3 "" H 8500 4150 50  0001 C CNN
 	1    8100 3850
@@
 $EndComp
 $Comp
-L Device:CP C_420
+L Device:CP C420
 U 1 1 AA736363
 P 4250 5250
-F 0 "C_420" V 4100 5200 50  0000 L CNN
+F 0 "C420" V 4100 5200 50  0000 L CNN
 F 1 "1µ/50v" V 4400 5150 50  0000 L CNN
-F 2 "" H 4288 5100 50  0001 C CNN
+F 2 "Capacitor_THT:CP_Radial_D4.0mm_P2.00mm" H 4288 5100 50  0001 C CNN
 F 3 "~" H 4250 5250 50  0001 C CNN
 	1    4250 5250
@@
 $EndComp
 $Comp
-L Device:CP C_430
+L Device:CP C430
 U 1 1 AA73661A
 P 7700 5450
-F 0 "C_430" H 7818 5496 50  0000 L CNN
+F 0 "C430" H 7818 5496 50  0000 L CNN
 F 1 "1µ/35vT" H 7818 5405 50  0000 L CNN
-F 2 "" H 7738 5300 50  0001 C CNN
+F 2 "Capacitor_THT:CP_Radial_D4.0mm_P2.00mm" H 7738 5300 50  0001 C CNN
 F 3 "~" H 7700 5450 50  0001 C CNN
 	1    7700 5450
@@
 $EndComp
 $Comp
-L Device:C C_421
+L Device:C C421
 U 1 1 AA736CC2
 P 2900 6500
-F 0 "C_421" H 3015 6546 50  0000 L CNN
+F 0 "C421" H 3015 6546 50  0000 L CNN
 F 1 "6n8" H 3015 6455 50  0000 L CNN
-F 2 "" H 2938 6350 50  0001 C CNN
+F 2 "Capacitor_SMD:C_0805_2012Metric_Pad1.18x1.45mm_HandSolder" H 2938 6350 50  0001 C CNN
 F 3 "~" H 2900 6500 50  0001 C CNN
+F 4 "C1755" H 2900 6500 50  0001 C CNN "LCSC"
 	1    2900 6500
 	1    0    0    -1
 $EndComp
 $Comp
-L Device:C C_533
+L Device:C C533
 U 1 1 AA737328
 P 8850 2200
-F 0 "C_533" H 8965 2246 50  0000 L CNN
+F 0 "C533" H 8900 2300 50  0000 L CNN
 F 1 "5n6" H 8965 2155 50  0000 L CNN
-F 2 "" H 8888 2050 50  0001 C CNN
+F 2 "Capacitor_SMD:C_0805_2012Metric_Pad1.18x1.45mm_HandSolder" H 8888 2050 50  0001 C CNN
 F 3 "~" H 8850 2200 50  0001 C CNN
+F 4 "C113862" H 8850 2200 50  0001 C CNN "LCSC"
 	1    8850 2200
 	1    0    0    -1
 $EndComp
 $Comp
-L Device:C C_530
+L Device:C C530
 U 1 1 AA7375C5
 P 3850 2000
-F 0 "C_530" V 3950 1700 50  0000 L CNN
+F 0 "C530" V 3950 1700 50  0000 L CNN
 F 1 "10n" V 3750 1750 50  0000 L CNN
-F 2 "" H 3888 1850 50  0001 C CNN
+F 2 "Capacitor_SMD:C_0805_2012Metric_Pad1.18x1.45mm_HandSolder" H 3888 1850 50  0001 C CNN
 F 3 "~" H 3850 2000 50  0001 C CNN
+F 4 "C1710" V 3850 2000 50  0001 C CNN "LCSC"
 	1    3850 2000
 	0    -1   -1   0
 $EndComp
 $Comp
-L Device:C C_531
+L Device:C C531
 U 1 1 AA73785B
 P 8200 2200
-F 0 "C_531" H 8315 2246 50  0000 L CNN
+F 0 "C531" H 8315 2246 50  0000 L CNN
 F 1 "6n8" H 8315 2155 50  0000 L CNN
-F 2 "" H 8238 2050 50  0001 C CNN
+F 2 "Capacitor_SMD:C_0805_2012Metric_Pad1.18x1.45mm_HandSolder" H 8238 2050 50  0001 C CNN
 F 3 "~" H 8200 2200 50  0001 C CNN
+F 4 "C1755" H 8200 2200 50  0001 C CNN "LCSC"
 	1    8200 2200
 	1    0    0    -1
 $EndComp
 $Comp
-L Device:R R_432
+L Device:R R432
 U 1 1 AA7393D6
 P 2250 6250
-F 0 "R_432" V 2350 6150 50  0000 L CNN
+F 0 "R432" V 2350 6150 50  0000 L CNN
 F 1 "3K3" V 2150 6200 50  0000 L CNN
-F 2 "" V 2180 6250 50  0001 C CNN
+F 2 "Resistor_SMD:R_0805_2012Metric_Pad1.20x1.40mm_HandSolder" V 2180 6250 50  0001 C CNN
 F 3 "~" H 2250 6250 50  0001 C CNN
+F 4 "C110574" V 2250 6250 50  0001 C CNN "LCSC"
 	1    2250 6250
 	0    -1   -1   0
 $EndComp
 $Comp
-L Device:R R_422
+L Device:R R422
 U 1 1 AA739868
 P 2900 6000
-F 0 "R_422" H 2970 6046 50  0000 L CNN
+F 0 "R422" H 2970 6046 50  0000 L CNN
 F 1 "8K2" H 2970 5955 50  0000 L CNN
-F 2 "" V 2830 6000 50  0001 C CNN
+F 2 "Resistor_SMD:R_0805_2012Metric_Pad1.20x1.40mm_HandSolder" V 2830 6000 50  0001 C CNN
 F 3 "~" H 2900 6000 50  0001 C CNN
+F 4 "C17828" H 2900 6000 50  0001 C CNN "LCSC"
 	1    2900 6000
 	1    0    0    -1
 $EndComp
 $Comp
-L Device:R R_531
+L Device:R R531
 U 1 1 AA739AEB
 P 8200 1650
-F 0 "R_531" V 8300 1550 50  0000 L CNN
+F 0 "R531" V 8300 1550 50  0000 L CNN
 F 1 "68K" V 8100 1600 50  0000 L CNN
-F 2 "" V 8130 1650 50  0001 C CNN
+F 2 "Resistor_SMD:R_0805_2012Metric_Pad1.20x1.40mm_HandSolder" V 8130 1650 50  0001 C CNN
 F 3 "~" H 8200 1650 50  0001 C CNN
+F 4 "C17801" V 8200 1650 50  0001 C CNN "LCSC"
 	1    8200 1650
 	0    -1   -1   0
 $EndComp
 $Comp
-L Device:R R_430
+L Device:R R430
 U 1 1 AA739D78
 P 9400 6250
-F 0 "R_430" V 9500 6150 50  0000 L CNN
+F 0 "R430" V 9500 6150 50  0000 L CNN
 F 1 "24K" V 9300 6150 50  0000 L CNN
-F 2 "" V 9330 6250 50  0001 C CNN
+F 2 "Resistor_SMD:R_0805_2012Metric_Pad1.20x1.40mm_HandSolder" V 9330 6250 50  0001 C CNN
 F 3 "~" H 9400 6250 50  0001 C CNN
+F 4 "C17575" V 9400 6250 50  0001 C CNN "LCSC"
 	1    9400 6250
 	0    1    -1   0
 $EndComp
 $Comp
-L Device:R R_532
+L Device:R R532
 U 1 1 AA739F78
 P 7350 1650
-F 0 "R_532" V 7250 1550 50  0000 L CNN
+F 0 "R532" V 7250 1550 50  0000 L CNN
 F 1 "6K8" V 7450 1600 50  0000 L CNN
-F 2 "" V 7280 1650 50  0001 C CNN
+F 2 "Resistor_SMD:R_0805_2012Metric_Pad1.20x1.40mm_HandSolder" V 7280 1650 50  0001 C CNN
 F 3 "~" H 7350 1650 50  0001 C CNN
+F 4 "C17772" V 7350 1650 50  0001 C CNN "LCSC"
 	1    7350 1650
 	0    1    1    0
 $EndComp
 $Comp
-L Device:CP C_532
+L Device:CP C532
 U 1 1 AA73CBBF
 P 6550 1650
-F 0 "C_532" V 6650 1350 50  0000 L CNN
+F 0 "C532" V 6650 1350 50  0000 L CNN
 F 1 "1µ/50v" V 6450 1250 50  0000 L CNN
-F 2 "" H 6588 1500 50  0001 C CNN
+F 2 "Capacitor_THT:CP_Radial_D4.0mm_P2.00mm" H 6588 1500 50  0001 C CNN
 F 3 "~" H 6550 1650 50  0001 C CNN
 	1    6550 1650
@@
 Text HLabel 10600 5750 2    50   Input ~ 0
 pin6_vsize
-Text HLabel 10700 4350 2    50   Output ~ 0
+Text HLabel 10800 4350 2    50   Output ~ 0
 pin7_vdrv
 Text HLabel 10600 6250 2    50   Input ~ 0
@@
 Text HLabel 1550 750  0    50   Input ~ 0
 pin10_prot
-Text HLabel 10700 3450 2    50   Output ~ 0
+Text HLabel 10750 3450 2    50   Output ~ 0
 pin11_hdrv
 Text HLabel 1550 1050 0    50   Input ~ 0
@@
 	8200 2350 8200 2400
 Wire Wire Line
-	5200 4750 3550 4750
+	5200 4750 4300 4750
 Connection ~ 5200 4750
 Wire Wire Line
@@
 Wire Wire Line
 	9100 1050 9100 2550
-Wire Wire Line
-	1550 5000 1700 5000
 NoConn ~ 1700 5000
 Wire Wire Line
@@
 Wire Wire Line
 	2900 2950 2900 5750
+$Comp
+L Device:C C533b1
+U 1 1 6A39B5B3
+P 9350 2200
+F 0 "C533b1" H 9400 2300 50  0000 L CNN
+F 1 "5n6" H 9465 2155 50  0000 L CNN
+F 2 "Capacitor_THT:C_Rect_L7.0mm_W3.5mm_P2.50mm_P5.00mm" H 9388 2050 50  0001 C CNN
+F 3 "~" H 9350 2200 50  0001 C CNN
+	1    9350 2200
+	1    0    0    -1
+$EndComp
+$Comp
+L power:GND #PWR0103
+U 1 1 6A39BAB8
+P 9350 2450
+F 0 "#PWR0103" H 9350 2200 50  0001 C CNN
+F 1 "GND" H 9355 2277 50  0000 C CNN
+F 2 "" H 9350 2450 50  0001 C CNN
+F 3 "" H 9350 2450 50  0001 C CNN
+	1    9350 2450
+	1    0    0    -1
+$EndComp
+Wire Wire Line
+	9350 2450 9350 2350
+Wire Wire Line
+	9350 2050 9350 1650
+Wire Wire Line
+	9350 1650 8850 1650
+Connection ~ 8850 1650
+$Comp
+L Connector:TestPoint TP1
+U 1 1 6A3B1DFC
+P 4300 4350
+F 0 "TP1" H 4358 4468 50  0000 L CNN
+F 1 "GND" H 4358 4377 50  0000 L CNN
+F 2 "TestPoint:TestPoint_Bridge_Pitch2.54mm_Drill1.0mm" H 4500 4350 50  0001 C CNN
+F 3 "~" H 4500 4350 50  0001 C CNN
+	1    4300 4350
+	1    0    0    -1
+$EndComp
+Wire Wire Line
+	4300 4350 4300 4750
+$Comp
+L Connector:TestPoint TP2
+U 1 1 6A3B4004
+P 10700 2700
+F 0 "TP2" H 10758 2818 50  0000 L CNN
+F 1 "H" H 10758 2727 50  0000 L CNN
+F 2 "TestPoint:TestPoint_Bridge_Pitch2.54mm_Drill1.0mm" H 10900 2700 50  0001 C CNN
+F 3 "~" H 10900 2700 50  0001 C CNN
+	1    10700 2700
+	1    0    0    -1
+$EndComp
+Wire Wire Line
+	10750 3450 10700 3450
+Wire Wire Line
+	10700 3450 10700 2700
+Connection ~ 10700 3450
+$Comp
+L Connector:TestPoint TP3
+U 1 1 6A3B7DCC
+P 10700 4200
+F 0 "TP3" H 10758 4318 50  0000 L CNN
+F 1 "V" H 10758 4227 50  0000 L CNN
+F 2 "TestPoint:TestPoint_Bridge_Pitch2.54mm_Drill1.0mm" H 10900 4200 50  0001 C CNN
+F 3 "~" H 10900 4200 50  0001 C CNN
+	1    10700 4200
+	1    0    0    -1
+$EndComp
+Wire Wire Line
+	10800 4350 10700 4350
+Wire Wire Line
+	10700 4350 10700 4200
+Connection ~ 10700 4350
+Wire Wire Line
+	1550 5000 1700 5000
+Connection ~ 4300 4750
+Wire Wire Line
+	4300 4750 3550 4750
 $EndSCHEMATC
