File: SHIC402.sch (KiCad schematic (older format))
At the start: 31 parts, among them IC2 M5223

Commit message: Some corrections
Parts:
- added H1: MountingHole, MountingHole:MountingHole_3.7mm, symbol Mechanical:MountingHole
- IC2: value M5223 -> 4558; footprint (none) -> Package_SO:SOIC-8_3.9x4.9mm_P1.27mm
- IC2: value M5223 -> 4558; footprint (none) -> Package_SO:SOIC-8_3.9x4.9mm_P1.27mm; LCSC (none) -> C6955
- _C1, _C2, _C3, _C4: footprint (none) -> Capacitor_THT:CP_Radial_D4.0mm_P2.00mm
- _D1: renamed from _D1_NP1; value 1N4148 -> 4148; footprint (none) -> Diode_SMD:D_SOD-323_HandSoldering; LCSC (none) -> C2128
- _D2: renamed from _Dxx1; value 1N4148 -> 4148; footprint (none) -> Diode_SMD:D_SOD-323_HandSoldering; LCSC (none) -> C2128
- _IC1: footprint (none) -> Package_SIP:SIP9_Housing_BigPads
- _Q1: value 2SC1740 -> MMBT3904; footprint Package_TO_SOT_THT:TO-92_Inline -> Package_TO_SOT_SMD:SOT-23; symbol Transistor_BJT:2SC1815 -> Transistor_BJT:MMBT3904; LCSC (none) -> C20526
- _R1, _R14, _R2, _R3, _R4, _R5, _R7: footprint (none) -> Resistor_SMD:R_0805_2012Metric_Pad1.20x1.40mm_HandSolder
- _R10: footprint (none) -> Resistor_SMD:R_0805_2012Metric_Pad1.20x1.40mm_HandSolder; LCSC (none) -> C17560
- _R11, _R12, _R13, _R18, _R19, _R20, _R21, _R6: footprint (none) -> Resistor_SMD:R_0805_2012Metric_Pad1.20x1.40mm_HandSolder; LCSC (none) -> C149504
- _R15, _R8: footprint (none) -> Resistor_SMD:R_0805_2012Metric_Pad1.20x1.40mm_HandSolder; LCSC (none) -> C17756
- _R16: renamed from _R18_NP1; footprint (none) -> Resistor_SMD:R_0805_2012Metric_Pad1.20x1.40mm_HandSolder; LCSC (none) -> C149504
- _R17: renamed from _R17_NP1; footprint (none) -> Resistor_SMD:R_0805_2012Metric_Pad1.20x1.40mm_HandSolder; LCSC (none) -> C149504
- _R9: footprint (none) -> Resistor_SMD:R_0805_2012Metric_Pad1.20x1.40mm_HandSolder; LCSC (none) -> C17840
- _VR1: footprint (none) -> _my:minipot
Connections:
- net labels added: pin6_hsize, pin7_spc
- net labels removed: pin6, pin7
- wire segments 92 -> 94
Other:
- note added: "(hsize)"
- note added: "(spc)"
- note added: "D1, R16, R17\nNOT POPULATED"
- note removed: "D1, R17, R18\nNOT POPULATED"
